Commit message: updates incorrect min/max position limits in the motor config files and urdfs

File: interbotix_ros_xsarms/interbotix_xsarm_descriptions/urdf/px150.urdf.xacro (robot description, xacro)
@@ -83,5 +83,5 @@
   <joint name="shoulder" type="revolute">
     <axis xyz="0 1 0"/>
-    <limit effort="18" lower="${radians(-111)}" upper="${radians(111)}" velocity="${pi}"/>
+    <limit effort="18" lower="${radians(-113)}" upper="${radians(111)}" velocity="${pi}"/>
     <origin rpy="0 0 0" xyz="0 0 0.03891"/>
     <parent link="$(arg robot_name)/shoulder_link"/>

File: interbotix_ros_xsarms/interbotix_xsarm_descriptions/urdf/rx200.urdf.xacro (robot description, xacro)
@@ -83,5 +83,5 @@
   <joint name="shoulder" type="revolute">
     <axis xyz="0 1 0"/>
-    <limit effort="18" lower="${radians(-107)}" upper="${radians(111)}" velocity="1"/>
+    <limit effort="18" lower="${radians(-108)}" upper="${radians(113)}" velocity="1"/>
     <origin rpy="0 0 0" xyz="0 0 0.03891"/>
     <parent link="$(arg robot_name)/shoulder_link"/>

File: interbotix_ros_xsarms/interbotix_xsarm_descriptions/urdf/vx300.urdf.xacro (robot description, xacro)
@@ -83,5 +83,5 @@
   <joint name="shoulder" type="revolute">
     <axis xyz="0 1 0"/>
-    <limit effort="20" lower="${radians(-106)}" upper="${radians(101)}" velocity="${pi}"/>
+    <limit effort="20" lower="${radians(-106)}" upper="${radians(72)}" velocity="${pi}"/>
     <origin rpy="0 0 0" xyz="0 0 0.04805"/>
     <parent link="$(arg robot_name)/shoulder_link"/>
@@ -157,5 +157,5 @@
   <joint name="wrist_angle" type="revolute">
     <axis xyz="0 1 0"/>
-    <limit effort="5" lower="${radians(-107)}" upper="${radians(130)}" velocity="${pi}"/>
+    <limit effort="5" lower="${radians(-107)}" upper="${radians(128)}" velocity="${pi}"/>
     <origin rpy="0 0 0" xyz="0.3 0 0"/>
     <parent link="$(arg robot_name)/forearm_link"/>

File: interbotix_ros_xsarms/interbotix_xsarm_descriptions/urdf/vx300s.urdf.xacro (robot description, xacro)
@@ -83,5 +83,5 @@
   <joint name="shoulder" type="revolute">
     <axis xyz="0 1 0"/>
-    <limit effort="20" lower="${radians(-106)}" upper="${radians(101)}" velocity="${pi}"/>
+    <limit effort="20" lower="${radians(-106)}" upper="${radians(72)}" velocity="${pi}"/>
     <origin rpy="0 0 0" xyz="0 0 0.04805"/>
     <parent link="$(arg robot_name)/shoulder_link"/>
@@ -194,5 +194,5 @@
   <joint name="wrist_angle" type="revolute">
     <axis xyz="0 1 0"/>
-    <limit effort="5" lower="${radians(-107)}" upper="${radians(130)}" velocity="${pi}"/>
+    <limit effort="5" lower="${radians(-107)}" upper="${radians(128)}" velocity="${pi}"/>
     <origin rpy="0 0 0" xyz="0.1 0 0"/>
     <parent link="$(arg robot_name)/lower_forearm_link"/>

File: interbotix_ros_xsarms/interbotix_xsarm_descriptions/urdf/wx200.urdf.xacro (robot description, xacro)
@@ -157,5 +157,5 @@
   <joint name="wrist_angle" type="revolute">
     <axis xyz="0 1 0"/>
-    <limit effort="5" lower="${radians(-123)}" upper="${radians(100)}" velocity="${pi}"/>
+    <limit effort="5" lower="${radians(-100)}" upper="${radians(123)}" velocity="${pi}"/>
     <origin rpy="0 0 0" xyz="0.2 0 0"/>
     <parent link="$(arg robot_name)/forearm_link"/>
