Commit message: Adjust joint positions and limits

File: interbotix_ros_xsarms/interbotix_xsarm_descriptions/urdf/wx200.urdf.xacro (robot description, xacro)
@@ -25,5 +25,5 @@
   <xacro:property name="waist_limit_vel"            value="${pi}"/>
   <xacro:property name="shoulder_limit_effort"      value="18"/>
-  <xacro:property name="shoulder_limit_lower"       value="${radians(-108)}"/>
+  <xacro:property name="shoulder_limit_lower"       value="${radians(-80)}"/>
   <xacro:property name="shoulder_limit_upper"       value="${radians(113)}"/>
   <xacro:property name="shoulder_limit_vel"         value="1"/>
