Commit message: Initial work to px100, interbotix_arm

File: interbotix_ros_xsarms/interbotix_xsarm_descriptions/urdf/ar_tag.urdf.xacro (robot description, xacro)
@@ -1,50 +1,50 @@
 <?xml version="1.0"?>
 <robot xmlns:xacro="http://ros.org/wiki/xacro">
-  <!-- If the AR tag is being used, then add the AR tag mount -->
-  <joint name="ar_tag" type="fixed">
-    <axis xyz="0 0 0"/>
-    <origin
-      rpy="0 0 0"
-      xyz="-0.017 0 0.04155"/>
-    <parent
-      link="$(arg robot_name)/ee_arm_link"/>
-    <child
-      link="$(arg robot_name)/ar_tag_link"/>
-  </joint>
-  <link name="$(arg robot_name)/ar_tag_link">
-    <visual>
-      <origin
-        rpy="0 0 0"
-        xyz="0 0 0"/>
-      <geometry>
-        <mesh
-          filename="${mesh_directory}/../ar_tag.stl"
-          scale="0.001 0.001 0.001"/>
-      </geometry>
-      <material name="interbotix_black"/>
-    </visual>
-    <collision>
-      <origin
-        rpy="0 0 0"
-        xyz="0 0 0"/>
-      <geometry>
-        <mesh
-          filename="${mesh_directory}/../ar_tag.stl"
-          scale="0.001 0.001 0.001"/>
-      </geometry>
-    </collision>
-    <inertial>
-      <origin
-        rpy="0 0 0"
-        xyz="0 0 -0.00315"/>
-      <mass value="0.016507"/>
-      <inertia
-        ixx="0.000003084"
-        ixy="0"
-        ixz="0"
-        iyy="0.000003084"
-        iyz="0"
-        izz="0.000006059"/>
-    </inertial>
-  </link>
+  <xacro:macro name="ar_tag" params="robot_name parent_link *origin">
+    <!-- If the AR tag is being used, then add the AR tag mount -->
+    <joint name="ar_tag" type="fixed">
+      <axis xyz="0 0 0"/>
+      <xacro:insert_block name="origin"/>
+      <parent
+        link="${parent_link}"/>
+      <child
+        link="$(arg robot_name)/ar_tag_link"/>
+    </joint>
+    <link name="$(arg robot_name)/ar_tag_link">
+      <visual>
+        <origin
+          rpy="0 0 0"
+          xyz="0 0 0"/>
+        <geometry>
+          <mesh
+            filename="${mesh_directory}/../ar_tag.stl"
+            scale="0.001 0.001 0.001"/>
+        </geometry>
+        <material name="interbotix_black"/>
+      </visual>
+      <collision>
+        <origin
+          rpy="0 0 0"
+          xyz="0 0 0"/>
+        <geometry>
+          <mesh
+            filename="${mesh_directory}/../ar_tag.stl"
+            scale="0.001 0.001 0.001"/>
+        </geometry>
+      </collision>
+      <inertial>
+        <origin
+          rpy="0 0 0"
+          xyz="0 0 -0.00315"/>
+        <mass value="0.016507"/>
+        <inertia
+          ixx="0.000003084"
+          ixy="0"
+          ixz="0"
+          iyy="0.000003084"
+          iyz="0"
+          izz="0.000006059"/>
+      </inertial>
+    </link>
+  </xacro:macro>
 </robot>

File: interbotix_ros_xsarms/interbotix_xsarm_descriptions/urdf/px100.urdf.xacro (robot description, xacro)
@@ -1,282 +1,107 @@
 <?xml version="1.0"?>
-<robot name="px100" xmlns:xacro="http://ros.org/wiki/xacro">
-  <xacro:property name="robot_model"
-    value="px100"
-    scope="global"/>
-  <xacro:property name="dof"
-    value="4"
-    scope="global"/>
-  <xacro:arg name="robot_name"                      default="${robot_model}"/>
-  <xacro:arg name="base_link_frame"                 default="base_link"/>
-  <xacro:arg name="use_gripper"                     default="true"/>
-  <xacro:arg name="show_ar_tag"                     default="false"/>
-  <xacro:arg name="show_gripper_bar"                default="true"/>
-  <xacro:arg name="show_gripper_fingers"            default="true"/>
-  <xacro:arg name="use_world_frame"                 default="false"/>
-  <xacro:arg name="external_urdf_loc"               default=""/>
-  <xacro:arg name="hardware_type"                   default="actual"/>
-  <xacro:property name="mesh_directory"             value="package://interbotix_xsarm_descriptions/meshes/${robot_model}_meshes"/>
-  <xacro:property name="urdf_loc"                   value="$(arg external_urdf_loc)"/>
-  <xacro:property name="hardware_type"              value="$(arg hardware_type)"/>
-  <xacro:property name="pi_offset"                  value="0.00001"/>
-  <xacro:property name="waist_limit_effort"         value="1"/>
-  <xacro:property name="waist_limit_lower"          value="${-pi + pi_offset}"/>
-  <xacro:property name="waist_limit_upper"          value="${pi - pi_offset}"/>
-  <xacro:property name="waist_limit_vel"            value="${pi}"/>
-  <xacro:property name="shoulder_limit_effort"      value="2"/>
-  <xacro:property name="shoulder_limit_lower"       value="${radians(-111)}"/>
-  <xacro:property name="shoulder_limit_upper"       value="${radians(107)}"/>
-  <xacro:property name="shoulder_limit_vel"         value="${pi}"/>
-  <xacro:property name="elbow_limit_effort"         value="2"/>
-  <xacro:property name="elbow_limit_lower"          value="${radians(-121)}"/>
-  <xacro:property name="elbow_limit_upper"          value="${radians(92)}"/>
-  <xacro:property name="elbow_limit_vel"            value="${pi}"/>
-  <xacro:property name="wrist_angle_limit_effort"   value="1"/>
-  <xacro:property name="wrist_angle_limit_lower"    value="${radians(-100)}"/>
-  <xacro:property name="wrist_angle_limit_upper"    value="${radians(123)}"/>
-  <xacro:property name="wrist_angle_limit_vel"      value="${pi}"/>
-  <xacro:property name="gripper_limit_vel"          value="${pi}"/>
-  <xacro:property name="finger_limit_effort"        value="5"/>
-  <xacro:property name="finger_limit_lower"         value="0.015"/>
-  <xacro:property name="finger_limit_upper"         value="0.037"/>
-  <xacro:property name="finger_limit_vel"           value="1"/>
-  <material name="interbotix_black">
-    <texture filename="package://interbotix_xsarm_descriptions/meshes/interbotix_black.png"/>
-  </material>
-  <xacro:if value="$(arg use_world_frame)">
-    <link name="world"/>
-    <joint name="fixed" type="fixed">
-      <parent
-        link="world"/>
-      <child
-        link="$(arg robot_name)/$(arg base_link_frame)"/>
-    </joint>
-  </xacro:if> <!-- use_world_frame -->
-  <link name="$(arg robot_name)/$(arg base_link_frame)">
-    <visual>
-      <origin
-        rpy="0 0 ${pi/2}"
-        xyz="0 0 0"/>
-      <geometry>
-        <mesh
-          filename="${mesh_directory}/base.stl"
-          scale="0.001 0.001 0.001"/>
-      </geometry>
-      <material name="interbotix_black"/>
-    </visual>
-    <collision>
-      <origin
-        rpy="0 0 ${pi/2}"
-        xyz="0 0 0"/>
-      <geometry>
-        <mesh
-          filename="${mesh_directory}/base.stl"
-          scale="0.001 0.001 0.001"/>
-      </geometry>
-    </collision>
-    <inertial>
-      <origin
-        rpy="0 0 ${pi/2}"
-        xyz="-0.0332053000 0.0008915770 0.0211913000"/>
-      <mass value="0.395887"/>
-      <inertia
-        ixx="0.0010650000"
-        iyy="0.0003332000"
-        izz="0.0012080000"
-        ixy="-0.0000130300"
-        ixz="0.0000018614"
-        iyz="0.0000409200"/>
-    </inertial>
-  </link>
-  <joint name="waist" type="revolute">
-    <axis xyz="0 0 1"/>
-    <limit
-      effort="${waist_limit_effort}"
-      lower="${waist_limit_lower}"
-      upper="${waist_limit_upper}"
-      velocity="${waist_limit_vel}"/>
-    <origin
-      rpy="0 0 0"
-      xyz="0 0 0.05085"/>
-    <parent
-      link="$(arg robot_name)/$(arg base_link_frame)"/>
-    <child
-      link="$(arg robot_name)/shoulder_link"/>
-    <dynamics
-      friction="0.1"
-      damping="0.1"/>
-  </joint>
-  <link name="$(arg robot_name)/shoulder_link">
-    <visual>
-      <origin
-        rpy="0 0 ${pi/2}"
-        xyz="0 0 -0.0022"/>
-      <geometry>
-        <mesh
-          filename="${mesh_directory}/shoulder.stl"
-          scale="0.001 0.001 0.001"/>
-      </geometry>
-      <material name="interbotix_black"/>
-    </visual>
-    <collision>
-      <origin
-        rpy="0 0 ${pi/2}"
-        xyz="0 0 -0.0022"/>
-      <geometry>
-        <mesh
-          filename="${mesh_directory}/shoulder.stl"
-          scale="0.001 0.001 0.001"/>
-      </geometry>
-    </collision>
-    <inertial>
-      <origin
-        rpy="0 0 ${pi/2}"
-        xyz="0.0000111169 -0.0003605640 0.0284598000"/>
-      <mass value="0.072587"/>
-      <inertia
-        ixx="0.0000231000"
-        iyy="0.0000253500"
-        izz="0.0000144200"
-        ixy="0.0000000003"
-        ixz="0.0000001606"
-        iyz="-0.0000000206"/>
-    </inertial>
-  </link>
-  <joint name="shoulder" type="revolute">
-    <axis xyz="0 1 0"/>
-    <limit
-      effort="${shoulder_limit_effort}"
-      lower="${shoulder_limit_lower}"
-      upper="${shoulder_limit_upper}"
-      velocity="${shoulder_limit_vel}"/>
-    <origin
-      rpy="0 0 0"
-      xyz="0 0 0.04225"/>
-    <parent
-      link="$(arg robot_name)/shoulder_link"/>
-    <child
-      link="$(arg robot_name)/upper_arm_link"/>
-    <dynamics
-      friction="0.1"
-      damping="0.1"/>
-  </joint>
-  <link name="$(arg robot_name)/upper_arm_link">
-    <visual>
-      <origin
-        rpy="0 0 ${pi/2}"
-        xyz="0 0 0"/>
-      <geometry>
-        <mesh
-          filename="${mesh_directory}/upper_arm.stl"
-          scale="0.001 0.001 0.001"/>
-      </geometry>
-      <material name="interbotix_black"/>
-    </visual>
-    <collision>
-      <origin
-        rpy="0 0 ${pi/2}"
-        xyz="0 0 0"/>
-      <geometry>
-        <mesh
-          filename="${mesh_directory}/upper_arm.stl"
-          scale="0.001 0.001 0.001"/>
-      </geometry>
-    </collision>
-    <inertial>
-      <origin
-        rpy="0 0 ${pi/2}"
-        xyz="0.0161976963 -0.0002929352 0.0877230000"/>
-      <mass value="0.082923"/>
-      <inertia
-        ixx="0.0000800600"
-        iyy="0.0000745900"
-        izz="0.0000368500"
-        ixy="-0.0000002144"
-        ixz="0.0000002982"
-        iyz="0.0000165700"/>
-    </inertial>
-  </link>
-  <joint name="elbow" type="revolute">
-    <axis xyz="0 1 0"/>
-    <limit
-      effort="${elbow_limit_effort}"
-      lower="${elbow_limit_lower}"
-      upper="${elbow_limit_upper}"
-      velocity="${elbow_limit_vel}"/>
-    <origin
-      rpy="0 0 0"
-      xyz="0.035 0 0.1"/>
-    <parent
-      link="$(arg robot_name)/upper_arm_link"/>
-    <child
-      link="$(arg robot_name)/forearm_link"/>
-    <dynamics
-      friction="0.1"
-      damping="0.1"/>
-  </joint>
-  <link name="$(arg robot_name)/forearm_link">
-    <visual>
-      <origin
-        rpy="0 0 ${pi/2}"
-        xyz="0 0 0"/>
-      <geometry>
-        <mesh
-          filename="${mesh_directory}/forearm.stl"
-          scale="0.001 0.001 0.001"/>
-      </geometry>
-      <material name="interbotix_black"/>
-    </visual>
-    <collision>
-      <origin
-        rpy="0 0 ${pi/2}"
-        xyz="0 0 0"/>
-      <geometry>
-        <mesh
-          filename="${mesh_directory}/forearm.stl"
-          scale="0.001 0.001 0.001"/>
-      </geometry>
-    </collision>
-    <inertial>
-      <origin
-        rpy="0 0 ${pi/2}"
-        xyz="0.0773720000 -0.0003324882 0.0000000000"/>
-      <mass value="0.073058"/>
-      <inertia
-        ixx="0.0000533800"
-        iyy="0.0000165300"
-        izz="0.0000603500"
-        ixy="-0.0000003073"
-        ixz="0.0000000000"
-        iyz="0.0000000000"/>
-    </inertial>
-  </link>
-  <!-- Include the gripper if used -->
-  <xacro:if value="$(arg use_gripper)">
-    <joint name="wrist_angle" type="revolute">
-      <axis xyz="0 1 0"/>
+<robot xmlns:xacro="http://ros.org/wiki/xacro">
+  <xacro:macro name="arm_macro" params="robot_name:=px100">
+    <xacro:property name="robot_model"
+      value="px100"/>
+    <xacro:property name="dof"
+      value="4"
+      scope="global"/>
+    <xacro:property name="mesh_directory"             value="package://interbotix_xsarm_descriptions/meshes/${robot_model}_meshes"/>
+    <xacro:property name="pi_offset"                  value="0.00001"/>
+    <xacro:property name="waist_limit_effort"         value="1"                   scope="parent"/>
+    <xacro:property name="waist_limit_lower"          value="${-pi + pi_offset}"  scope="parent"/>
+    <xacro:property name="waist_limit_upper"          value="${pi - pi_offset}"   scope="parent"/>
+    <xacro:property name="waist_limit_vel"            value="${pi}"               scope="parent"/>
+    <xacro:property name="shoulder_limit_effort"      value="2"                   scope="parent"/>
+    <xacro:property name="shoulder_limit_lower"       value="${radians(-111)}"    scope="parent"/>
+    <xacro:property name="shoulder_limit_upper"       value="${radians(107)}"     scope="parent"/>
+    <xacro:property name="shoulder_limit_vel"         value="${pi}"               scope="parent"/>
+    <xacro:property name="elbow_limit_effort"         value="2"                   scope="parent"/>
+    <xacro:property name="elbow_limit_lower"          value="${radians(-121)}"    scope="parent"/>
+    <xacro:property name="elbow_limit_upper"          value="${radians(92)}"      scope="parent"/>
+    <xacro:property name="elbow_limit_vel"            value="${pi}"               scope="parent"/>
+    <xacro:property name="wrist_angle_limit_effort"   value="1"                   scope="parent"/>
+    <xacro:property name="wrist_angle_limit_lower"    value="${radians(-100)}"    scope="parent"/>
+    <xacro:property name="wrist_angle_limit_upper"    value="${radians(123)}"     scope="parent"/>
+    <xacro:property name="wrist_angle_limit_vel"      value="${pi}"               scope="parent"/>
+    <xacro:property name="gripper_limit_vel"          value="${pi}"               scope="parent"/>
+    <xacro:property name="finger_limit_effort"        value="5"                   scope="parent"/>
+    <xacro:property name="finger_limit_lower"         value="0.015"               scope="parent"/>
+    <xacro:property name="finger_limit_upper"         value="0.037"               scope="parent"/>
+    <xacro:property name="finger_limit_vel"           value="1"                   scope="parent"/>
+    <material name="interbotix_black">
+      <texture filename="package://interbotix_xsarm_descriptions/meshes/interbotix_black.png"/>
+    </material>
+    <xacro:if value="$(arg use_world_frame)">
+      <link name="world"/>
+      <joint name="fixed" type="fixed">
+        <parent
+          link="world"/>
+        <child
+          link="${robot_name}/$(arg base_link_frame)"/>
+      </joint>
+    </xacro:if> <!-- use_world_frame -->
+    <link name="${robot_name}/$(arg base_link_frame)">
+      <visual>
+        <origin
+          rpy="0 0 ${pi/2}"
+          xyz="0 0 0"/>
+        <geometry>
+          <mesh
+            filename="${mesh_directory}/base.stl"
+            scale="0.001 0.001 0.001"/>
+        </geometry>
+        <material name="interbotix_black"/>
+      </visual>
+      <collision>
+        <origin
+          rpy="0 0 ${pi/2}"
+          xyz="0 0 0"/>
+        <geometry>
+          <mesh
+            filename="${mesh_directory}/base.stl"
+            scale="0.001 0.001 0.001"/>
+        </geometry>
+      </collision>
+      <inertial>
+        <origin
+          rpy="0 0 ${pi/2}"
+          xyz="-0.0332053000 0.0008915770 0.0211913000"/>
+        <mass value="0.395887"/>
+        <inertia
+          ixx="0.0010650000"
+          iyy="0.0003332000"
+          izz="0.0012080000"
+          ixy="-0.0000130300"
+          ixz="0.0000018614"
+          iyz="0.0000409200"/>
+      </inertial>
+    </link>
+    <joint name="waist" type="revolute">
+      <axis xyz="0 0 1"/>
       <limit
-        effort="${wrist_angle_limit_effort}"
-        lower="${wrist_angle_limit_lower}"
-        upper="${wrist_angle_limit_upper}"
-        velocity="${wrist_angle_limit_vel}"/>
+        effort="${waist_limit_effort}"
+        lower="${waist_limit_lower}"
+        upper="${waist_limit_upper}"
+        velocity="${waist_limit_vel}"/>
       <origin
         rpy="0 0 0"
-        xyz="0.1 0 0"/>
+        xyz="0 0 0.05085"/>
       <parent
-        link="$(arg robot_name)/forearm_link"/>
+        link="${robot_name}/$(arg base_link_frame)"/>
       <child
-        link="$(arg robot_name)/gripper_link"/>
+        link="${robot_name}/shoulder_link"/>
       <dynamics
         friction="0.1"
         damping="0.1"/>
     </joint>
-    <link name="$(arg robot_name)/gripper_link">
+    <link name="${robot_name}/shoulder_link">
       <visual>
         <origin
           rpy="0 0 ${pi/2}"
-          xyz="0 0 0"/>
-        <geometry>
-          <mesh
-            filename="${mesh_directory}/gripper.stl"
+          xyz="0 0 -0.0022"/>
+        <geometry>
+          <mesh
+            filename="${mesh_directory}/shoulder.stl"
             scale="0.001 0.001 0.001"/>
         </geometry>
@@ -286,8 +111,8 @@
         <origin
           rpy="0 0 ${pi/2}"
-          xyz="0 0 0"/>
-        <geometry>
-          <mesh
-            filename="${mesh_directory}/gripper.stl"
+          xyz="0 0 -0.0022"/>
+        <geometry>
+          <mesh
+            filename="${mesh_directory}/shoulder.stl"
             scale="0.001 0.001 0.001"/>
         </geometry>
@@ -296,61 +121,41 @@
         <origin
           rpy="0 0 ${pi/2}"
-          xyz="0.0446910000 0.0000000000 0.0113540000"/>
-        <mass value="0.069929"/>
+          xyz="0.0000111169 -0.0003605640 0.0284598000"/>
+        <mass value="0.072587"/>
         <inertia
-          ixx="0.0000226800"
-          iyy="0.0000204400"
-          izz="0.0000197400"
-          ixy="0.0000000000"
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