Commit message: [xsarm_descriptions] Fix control joint order
Move forearm_roll joint to its corrent sequence position.

Fixes #32

File: interbotix_ros_xsarms/interbotix_xsarm_descriptions/urdf/control.urdf.xacro (robot description, xacro)
@@ -41,4 +41,13 @@
       <state_interface name="position"/>
     </joint>
+    <xacro:if value="${dof >= 6}">
+      <joint name="forearm_roll">
+        <command_interface name="position">
+          <param name="min">"${forearm_roll_limit_lower}"</param>
+          <param name="max">"${forearm_roll_limit_upper}"</param>
+        </command_interface>
+        <state_interface name="position"/>
+      </joint>
+    </xacro:if>
     <joint name="wrist_angle">
       <command_interface name="position">
@@ -51,15 +60,6 @@
       <joint name="wrist_rotate">
         <command_interface name="position">
-            <param name="min">"${wrist_rotate_limit_lower}"</param>
-            <param name="max">"${wrist_rotate_limit_upper}"</param>
-        </command_interface>
-        <state_interface name="position"/>
-      </joint>
-    </xacro:if>
-    <xacro:if value="${dof >= 6}">
-      <joint name="forearm_roll">
-        <command_interface name="position">
-            <param name="min">"${forearm_roll_limit_lower}"</param>
-            <param name="max">"${forearm_roll_limit_upper}"</param>
+          <param name="min">"${wrist_rotate_limit_lower}"</param>
+          <param name="max">"${wrist_rotate_limit_upper}"</param>
         </command_interface>
         <state_interface name="position"/>

Commit message: WIP: MiV arm description and MoveIt configs
# Conflicts:
#	interbotix_ros_xsarms/interbotix_xsarm_descriptions/meshes/miv_arm_meshes/base.stl
#	interbotix_ros_xsarms/interbotix_xsarm_descriptions/meshes/miv_arm_meshes/gripper.stl
#	interbotix_ros_xsarms/interbotix_xsarm_descriptions/meshes/miv_arm_meshes/lower_forearm.stl
#	interbotix_ros_xsarms/interbotix_xsarm_descriptions/meshes/miv_arm_meshes/shoulder.stl
#	interbotix_ros_xsarms/interbotix_xsarm_descriptions/meshes/miv_arm_meshes/upper_arm.stl
#	interbotix_ros_xsarms/interbotix_xsarm_descriptions/meshes/miv_arm_meshes/upper_forearm.stl
#	interbotix_ros_xsarms/interbotix_xsarm_descriptions/meshes/miv_arm_meshes/wrist.stl

File: interbotix_ros_xsarms/interbotix_xsarm_descriptions/urdf/control.urdf.xacro (robot description, xacro)
@@ -13,5 +13,5 @@
       <!-- If doing basic simulation of the robot -->
       <xacro:if value="${hardware_type == 'fake'}">
-        <plugin>fake_components/GenericSystem</plugin>
+        <plugin>mock_components/GenericSystem</plugin>
       </xacro:if>
       <!-- If simulating the robot in Gazebo Classic -->

File: interbotix_ros_xsarms/interbotix_xsarm_descriptions/urdf/miv_arm.urdf.xacro (robot description, xacro)
@@ -7,10 +7,34 @@
     value="6"
     scope="global"/>
+  <xacro:property name="l1"
+    value="0.07775"
+    scope="global"/>
+  <xacro:property name="l2"
+    value="0.05675"
+    scope="global"/>
+  <xacro:property name="l3"
+    value="0.250"
+    scope="global"/>
+  <xacro:property name="l4"
+    value="0.0575"
+    scope="global"/>
+  <xacro:property name="l5"
+    value="0.150"
+    scope="global"/>
+  <xacro:property name="l6"
+    value="0.100"
+    scope="global"/>
+  <xacro:property name="l7"
+    value="0.065"
+    scope="global"/>
+  <xacro:property name="l8"
+    value="0.081"
+    scope="global"/>
   <xacro:arg name="robot_name"                      default="${robot_model}"/>
   <xacro:arg name="base_link_frame"                 default="base_link"/>
-  <xacro:arg name="use_gripper"                     default="true"/>
+  <xacro:arg name="use_gripper"                     default="false"/>
   <xacro:arg name="show_ar_tag"                     default="false"/>
-  <xacro:arg name="show_gripper_bar"                default="true"/>
-  <xacro:arg name="show_gripper_fingers"            default="true"/>
+  <xacro:arg name="show_gripper_bar"                default="false"/>
+  <xacro:arg name="show_gripper_fingers"            default="false"/>
   <xacro:arg name="use_world_frame"                 default="false"/>
   <xacro:arg name="external_urdf_loc"               default=""/>
@@ -106,5 +130,5 @@
     <origin
       rpy="0 0 0"
-      xyz="0 0 0.079"/>
+      xyz="0 0 ${l1}"/>
     <parent
       link="$(arg robot_name)/$(arg base_link_frame)"/>
@@ -119,5 +143,5 @@
       <origin
         rpy="0 0 ${pi/2}"
-        xyz="0 0 -0.003"/>
+        xyz="0 0 0"/>
       <geometry>
         <mesh
@@ -130,5 +154,5 @@
       <origin
         rpy="0 0 ${pi/2}"
-        xyz="0 0 -0.003"/>
+        xyz="0 0 0"/>
       <geometry>
         <mesh
@@ -160,5 +184,5 @@
     <origin
       rpy="0 0 0"
-      xyz="0 0 0.04805"/>
+      xyz="0 0 ${l2}"/>
     <parent
       link="$(arg robot_name)/shoulder_link"/>
@@ -214,5 +238,5 @@
     <origin
       rpy="0 0 0"
-      xyz="0.05955 0 0.3"/>
+      xyz="${l4} 0 ${l3}"/>
     <parent
       link="$(arg robot_name)/upper_arm_link"/>
@@ -268,5 +292,5 @@
     <origin
       rpy="0 0 0"
-      xyz="0.2 0 0"/>
+      xyz="${l5} 0 0"/>
     <parent
       link="$(arg robot_name)/upper_forearm_link"/>
@@ -322,5 +346,5 @@
     <origin
       rpy="0 0 0"
-      xyz="0.1 0 0"/>
+      xyz="${l6} 0 0"/>
     <parent
       link="$(arg robot_name)/lower_forearm_link"/>
@@ -378,5 +402,5 @@
       <origin
         rpy="0 0 0"
-        xyz="0.069744 0 0"/>
+        xyz="${l7} 0 0"/>
       <parent
         link="$(arg robot_name)/wrist_link"/>
@@ -391,5 +415,5 @@
         <origin
           rpy="0 0 ${pi/2}"
-          xyz="-0.02 0 0"/>
+          xyz="0 0 0"/>
         <geometry>
           <mesh
@@ -402,5 +426,5 @@
         <origin
           rpy="0 0 ${pi/2}"
-          xyz="-0.02 0 0"/>
+          xyz="0 0 0"/>
         <geometry>
           <mesh
@@ -427,5 +451,5 @@
       <origin
         rpy="0 0 0"
-        xyz="0.042825 0 0"/>
+        xyz="${l8} 0 0"/>
       <parent
         link="$(arg robot_name)/gripper_link"/>
