Commit message: [URDF] Added joint limits (commented)

File: interbotix_ros_xscobots/interbotix_xscobot_descriptions/urdf/control.urdf.xacro (robot description, xacro)
@@ -22,6 +22,6 @@
     <joint name="j1">
       <command_interface name="position">
-        <!-- <param name="min">"${waist_limit_lower}"</param>
-        <param name="max">"${waist_limit_upper}"</param> -->
+        <!-- <param name="min">"${j1_limit_lower}"</param>
+        <param name="max">"${j1_limit_upper}"</param> -->
       </command_interface>
       <state_interface name="position"/>
@@ -29,6 +29,6 @@
     <joint name="j2">
       <command_interface name="position">
-        <!-- <param name="min">"${shoulder_limit_lower}"</param>
-        <param name="max">"${shoulder_limit_upper}"</param> -->
+        <!-- <param name="min">"${j2_limit_lower}"</param>
+        <param name="max">"${j2_limit_upper}"</param> -->
       </command_interface>
       <state_interface name="position"/>
@@ -36,6 +36,6 @@
     <joint name="j3">
       <command_interface name="position">
-        <!-- <param name="min">"${elbow_limit_lower}"</param>
-        <param name="max">"${elbow_limit_upper}"</param> -->
+        <!-- <param name="min">"${j3_limit_lower}"</param>
+        <param name="max">"${j3_limit_upper}"</param> -->
       </command_interface>
       <state_interface name="position"/>
@@ -43,6 +43,6 @@
     <joint name="j4">
     <command_interface name="position">
-        <!-- <param name="min">"${forearm_roll_limit_lower}"</param>
-        <param name="max">"${forearm_roll_limit_upper}"</param> -->
+        <!-- <param name="min">"${j4_limit_lower}"</param>
+        <param name="max">"${j4_limit_upper}"</param> -->
     </command_interface>
     <state_interface name="position"/>
@@ -50,6 +50,6 @@
     <joint name="j5">
       <command_interface name="position">
-        <!-- <param name="min">"${wrist_angle_limit_lower}"</param>
-        <param name="max">"${wrist_angle_limit_upper}"</param> -->
+        <!-- <param name="min">"${j5_limit_lower}"</param> -->
+        <!-- <param name="max">"${j5_limit_upper}"</param> -->
       </command_interface>
       <state_interface name="position"/>
@@ -57,6 +57,6 @@
     <joint name="j6">
     <command_interface name="position">
-        <!-- <param name="min">"${wrist_rotate_limit_lower}"</param>
-        <param name="max">"${wrist_rotate_limit_upper}"</param> -->
+        <!-- <param name="min">"${j6_limit_lower}"</param>
+        <param name="max">"${j6_limit_upper}"</param> -->
     </command_interface>
     <state_interface name="position"/>
@@ -72,6 +72,6 @@
         <joint name="left_finger">
           <command_interface name="position">
-            <!-- <param name="min">"${finger_limit_lower}"</param>
-            <param name="max">"${-finger_limit_lower}"</param> -->
+            <!-- <param name="min">"${finger_limit_lower}"</param> -->
+            <!-- <param name="max">"${-finger_limit_lower}"</param> -->
           </command_interface>
           <state_interface name="position"/>
@@ -82,6 +82,6 @@
             <param name="multiplier">1</param> -->
             <command_interface name="position">
-              <!-- <param name="min">"${-finger_limit_lower}"</param>
-              <param name="max">"${finger_limit_lower}"</param> -->
+              <!-- <param name="min">"${-finger_limit_lower}"</param> -->
+              <!-- <param name="max">"${finger_limit_lower}"</param> -->
             </command_interface>
             <state_interface name="position"/>

File: interbotix_ros_xscobots/interbotix_xscobot_descriptions/urdf/dx400.urdf.xacro (robot description, xacro)
@@ -20,8 +20,21 @@
   <xacro:arg name="external_urdf_loc"     default=""/>
   <xacro:arg name="load_gazebo_configs"   default="false"/>
+  <xacro:arg name="hardware_type"         default="actual"/>
   <xacro:property name="mesh_directory"   value="package://interbotix_xscobot_descriptions/meshes/${robot_model}_meshes"/>
   <xacro:property name="urdf_loc"         value="$(arg external_urdf_loc)"/>
   <xacro:property name="hardware_type"    value="$(arg hardware_type)"/>
   <xacro:property name="pi_offset"        value="0.00001"/>
+  <xacro:property name="j1_limit_lower"        value="-6.70001"/>
+  <xacro:property name="j1_limit_upper"        value="0.00001"/>
+  <xacro:property name="j2_limit_lower"        value="-1.88001"/>
+  <xacro:property name="j2_limit_upper"        value="1.88001"/>
+  <xacro:property name="j3_limit_lower"        value="-2.70001"/>
+  <xacro:property name="j3_limit_upper"        value="2.70001"/>
+  <xacro:property name="j4_limit_lower"        value="-3.66001"/>
+  <xacro:property name="j4_limit_upper"        value="1.55001"/>
+  <xacro:property name="j5_limit_lower"        value="-4.00001"/>
+  <xacro:property name="j5_limit_upper"        value="1.60001"/>
+  <xacro:property name="j6_limit_lower"        value="-5.00001"/>
+  <xacro:property name="j6_limit_upper"        value="1.60001"/>
   <xacro:if value="$(arg load_gazebo_configs)">
     <xacro:include filename="$(find interbotix_common_sim)/textures/interbotix_texture.gazebo"/>
