Commit message: [xscobot_descriptions] WIP refine URDF
Create proper URDF except for inertial values. Add meshes.

File: interbotix_ros_xscobots/interbotix_xscobot_descriptions/urdf/dx400.urdf.xacro (robot description, xacro)
@@ -1,4 +1,10 @@
 <?xml version="1.0"?>
 <robot name="dx400" xmlns:xacro="http://ros.org/wiki/xacro">
+  <xacro:property name="robot_model"
+    value="dx400"
+    scope="global"/>
+  <xacro:property name="dof"
+    value="6"
+    scope="global"/>
   <xacro:arg name="robot_name"            default="dx400"/>
   <xacro:arg name="base_link_frame"       default="base_link"/>
@@ -14,221 +20,530 @@
   <xacro:arg name="external_urdf_loc"     default=""/>
   <xacro:arg name="load_gazebo_configs"   default="false"/>
-  <xacro:property name="urdf_loc" value="$(arg external_urdf_loc)"/>
-  <xacro:property name="pi_offset" value="0.00001"/>
+  <xacro:property name="mesh_directory"   value="package://interbotix_xscobot_descriptions/meshes/${robot_model}_meshes"/>
+  <xacro:property name="urdf_loc"         value="$(arg external_urdf_loc)"/>
+  <xacro:property name="hardware_type"    value="$(arg hardware_type)"/>
+  <xacro:property name="pi_offset"        value="0.00001"/>
   <xacro:if value="$(arg load_gazebo_configs)">
     <xacro:include filename="$(find interbotix_common_sim)/textures/interbotix_texture.gazebo"/>
   </xacro:if>
   <material name="interbotix_black">
-    <color rgba="${220/255} ${220/255} ${220/255} 0.2"/>
-    <!-- <texture filename="package://interbotix_common_sim/media/materials/textures/interbotix_black.png"/> -->
+    <!-- <color rgba="${220/255} ${220/255} ${220/255} 0.2"/> -->
+    <texture filename="package://interbotix_common_sim/media/materials/textures/interbotix_black.png"/>
   </material>
   <xacro:if value="$(arg use_world_frame)">
     <link name="world"/>
     <joint name="fixed" type="fixed">
-      <parent link="world"/>
-      <child link="$(arg robot_name)/$(arg base_link_frame)"/>
+      <parent
+        link="world"/>
+      <child
+        link="$(arg robot_name)/$(arg base_link_frame)"/>
     </joint>
   </xacro:if>
   <link name="$(arg robot_name)/$(arg base_link_frame)">
-    <inertial>
-      <origin rpy="0 0 0" xyz="0 0 0"/>
-      <mass value="0.1" />
-      <inertia ixx="0.0" iyy="0.0" izz="0.0" ixy="0.0" ixz="0.0" iyz="0.0" />
-    </inertial>
+    <visual>
+      <origin
+        rpy="0 0 0"
+        xyz="0 0 0"/>
+      <geometry>
+        <mesh
+          filename="${mesh_directory}/base_link.stl"
+          scale="1 1 1"/>
+      </geometry>
+      <material name="interbotix_black"/>
+    </visual>
+    <inertial>
+      <origin
+        rpy="0 0 0"
+        xyz="0 0 0"/>
+      <mass value="0.1"/>
+      <inertia
+        ixx="4.18E-03"
+        iyy="4.44E-03"
+        izz="5.07E-03"
+        ixy="1.24E-05"
+        ixz="6.61E-05"
+        iyz="-1.88E-06"/>
+    </inertial>
+    <collision>
+      <origin
+        rpy="0 0 0"
+        xyz="0 0 0"/>
+      <geometry>
+        <mesh
+          filename="${mesh_directory}/base_link.stl"
+          scale="1 1 1"/>
+      </geometry>
+      <material name="interbotix_black"/>
+    </collision>
   </link>
   <joint name="j1" type="revolute">
     <axis xyz="0 0 1"/>
-    <limit effort="10" lower="${-pi + pi_offset}" upper="${pi - pi_offset}" velocity="${pi}"/>
-    <origin rpy="0 0 0" xyz="0 0 0.056"/>
-    <parent link="$(arg robot_name)/$(arg base_link_frame)"/>
-    <child link="$(arg robot_name)/link_1"/>
-    <dynamics friction="0.1"/>
-  </joint>
-  <transmission name="trans_j1">
-    <type>transmission_interface/SimpleTransmission</type>
-    <joint name="j1">
-      <hardwareInterface>hardware_interface/EffortJointInterface</hardwareInterface>
-    </joint>
-    <actuator name="j1_motor">
-      <mechanicalReduction>1</mechanicalReduction>
-    </actuator>
-  </transmission>
+    <limit
+      effort="10"
+      lower="${-pi + pi_offset}"
+      upper="${pi - pi_offset}"
+      velocity="${pi}"/>
+    <origin
+      rpy="0 0 0"
+      xyz="0 0 0"/>
+    <parent
+      link="$(arg robot_name)/$(arg base_link_frame)"/>
+    <child
+      link="$(arg robot_name)/link_1"/>
+    <dynamics
+      friction="0.1"
+      damping="0.1"/>
+  </joint>
   <link name="$(arg robot_name)/link_1">
-    <inertial>
-      <origin rpy="0 0 0" xyz="0.0 0.0 0.0"/>
-      <mass value="0.1" />
-      <inertia ixx="0.0" iyy="0.0" izz="0.0" ixy="0.0" ixz="0.0" iyz="0.0" />
-    </inertial>
+    <visual>
+      <origin
+        rpy="0 0 0"
+        xyz="0 0 0"/>
+      <geometry>
+        <mesh
+          filename="${mesh_directory}/link_1.stl"
+          scale="1 1 1"/>
+      </geometry>
+      <material name="interbotix_black"/>
+    </visual>
+    <inertial>
+      <origin
+        rpy="0 0 0"
+        xyz="0 0 0"/>
+      <mass value="0.1"/>
+      <inertia
+        ixx="0.0"
+        iyy="0.0"
+        izz="0.0"
+        ixy="0.0"
+        ixz="0.0"
+        iyz="0.0"/>
+    </inertial>
+    <collision>
+      <origin
+        rpy="0 0 0"
+        xyz="0 0 0"/>
+      <geometry>
+        <mesh
+          filename="${mesh_directory}/link_1.stl"
+          scale="1 1 1"/>
+      </geometry>
+      <material name="interbotix_black"/>
+    </collision>
   </link>
   <joint name="j2" type="revolute">
-    <axis xyz="0 -1 0"/>
-    <limit effort="10" lower="${-pi + pi_offset}" upper="${pi - pi_offset}" velocity="${pi}"/>
-    <!-- <limit effort="20" lower="${radians(-109)}" upper="${radians(109)}" velocity="${pi}"/> -->
-    <origin rpy="0 0 0" xyz="0 0.055 0.069288"/>
-    <parent link="$(arg robot_name)/link_1"/>
-    <child link="$(arg robot_name)/link_2"/>
-    <dynamics friction="0.1"/>
-  </joint>
-  <transmission name="trans_j2">
-    <type>transmission_interface/SimpleTransmission</type>
-    <joint name="j2">
-      <hardwareInterface>hardware_interface/EffortJointInterface</hardwareInterface>
-    </joint>
-    <actuator name="j2_motor">
-      <mechanicalReduction>1</mechanicalReduction>
-    </actuator>
-  </transmission>
+    <axis xyz="0 1 0"/>
+    <limit
+      effort="10"
+      lower="${-pi + pi_offset}"
+      upper="${pi - pi_offset}"
+      velocity="${pi}"/>
+    <origin
+      rpy="0 0 0"
+      xyz="0 0.055 0.119787"/>
+    <parent
+      link="$(arg robot_name)/link_1"/>
+    <child
+      link="$(arg robot_name)/link_2"/>
+    <dynamics
+      friction="0.1"
+      damping="0.1"/>
+  </joint>
   <link name="$(arg robot_name)/link_2">
-    <inertial>
-      <origin rpy="0 0 0" xyz="0.0 0.0 0.0"/>
-      <mass value="0.1" />
-      <inertia ixx="0.0" iyy="0.0" izz="0.0" ixy="-0.0" ixz="-0.0" iyz="0.0" />
-    </inertial>
+    <visual>
+      <origin
+        rpy="0 0 0"
+        xyz="0 0 0"/>
+      <geometry>
+        <mesh
+          filename="${mesh_directory}/link_2.stl"
+          scale="1 1 1"/>
+      </geometry>
+      <material name="interbotix_black"/>
+    </visual>
+    <inertial>
+      <origin
+        rpy="0 0 0"
+        xyz="0.0 0.0 0.0"/>
+      <mass value="0.1"/>
+      <inertia
+        ixx="0.0"
+        iyy="0.0"
+        izz="0.0"
+        ixy="-0.0"
+        ixz="-0.0"
+        iyz="0.0"/>
+    </inertial>
+    <collision>
+      <origin
+        rpy="0 0 0"
+        xyz="0 0 0"/>
+      <geometry>
+        <mesh
+          filename="${mesh_directory}/link_2.stl"
+          scale="1 1 1"/>
+      </geometry>
+      <material name="interbotix_black"/>
+    </collision>
   </link>
   <joint name="j3" type="revolute">
-    <axis xyz="0 -1 0"/>
-    <limit effort="10" lower="${-pi + pi_offset}" upper="${pi - pi_offset}" velocity="${pi}"/>
-    <!-- <limit effort="15" lower="${radians(-175)}" upper="${radians(175)}" velocity="${pi}"/> -->
-    <origin rpy="0 0 0" xyz="0 0 0.2285"/>
-    <parent link="$(arg robot_name)/link_2"/>
-    <child link="$(arg robot_name)/link_3"/>
-    <dynamics friction="0.1"/>
-  </joint>
-  <transmission name="trans_elbow">
-    <type>transmission_interface/SimpleTransmission</type>
-    <joint name="j3">
-      <hardwareInterface>hardware_interface/EffortJointInterface</hardwareInterface>
-    </joint>
-    <actuator name="elbow_motor">
-      <mechanicalReduction>1</mechanicalReduction>
-    </actuator>
-  </transmission>
+    <axis xyz="0 1 0"/>
+    <limit
+      effort="10"
+      lower="${-pi + pi_offset}"
+      upper="${pi - pi_offset}"
+      velocity="${pi}"/>
+    <origin
+      rpy="0 0 0"
+      xyz="0 -0.0248 0.17"/>
+    <parent
+      link="$(arg robot_name)/link_2"/>
+    <child
+      link="$(arg robot_name)/link_3"/>
+    <dynamics
+      friction="0.1"
+      damping="0.1"/>
+  </joint>
   <link name="$(arg robot_name)/link_3">
-    <inertial>
-      <origin rpy="0 0 0" xyz="0.0 0.0 0.0"/>
-      <mass value="0.1" />
-      <inertia ixx="0.0" iyy="0.0" izz="0.0" ixy="0.0" ixz="0" iyz="0" />
-    </inertial>
+    <visual>
+      <origin
+        rpy="0 0 ${pi}"
+        xyz="0 0 0"/>
+      <geometry>
+        <mesh
+          filename="${mesh_directory}/link_3.stl"
+          scale="1 1 1"/>
+      </geometry>
+      <material name="interbotix_black"/>
+    </visual>
+    <inertial>
+      <origin
+        rpy="0 0 0"
+        xyz="0.0 0.0 0.0"/>
+      <mass value="0.1"/>
+      <inertia
+        ixx="0.0"
+        iyy="0.0"
+        izz="0.0"
+        ixy="0.0"
+        ixz="0"
+        iyz="0"/>
+    </inertial>
+    <collision>
+      <origin
+        rpy="0 0 ${pi}"
+        xyz="0 0 0"/>
+      <geometry>
+        <mesh
+          filename="${mesh_directory}/link_3.stl"
+          scale="1 1 1"/>
+      </geometry>
+      <material name="interbotix_black"/>
+    </collision>
   </link>
   <joint name="j4" type="revolute">
     <axis xyz="0 1 0"/>
-    <limit effort="10" lower="${-pi + pi_offset}" upper="${pi - pi_offset}" velocity="${pi}"/>
-    <!-- <limit effort="2" lower="${radians(-172)}" upper="${radians(91)}" velocity="${pi}"/> -->
-    <origin rpy="0 0 0" xyz="0 -0.0541 0.20889"/>
-    <parent link="$(arg robot_name)/link_3"/>
-    <child link="$(arg robot_name)/link_4"/>
-    <dynamics friction="0.1"/>
-  </joint>
-  <transmission name="trans_forearm_roll">
-    <type>transmission_interface/SimpleTransmission</type>
-    <joint name="j4">
-      <hardwareInterface>hardware_interface/EffortJointInterface</hardwareInterface>
-    </joint>
-    <actuator name="forearm_roll_motor">
-      <mechanicalReduction>1</mechanicalReduction>
-    </actuator>
-  </transmission>
+    <limit
+      effort="10"
+      lower="${-pi + pi_offset}"
+      upper="${pi - pi_offset}"
+      velocity="${pi}"/>
+    <origin
+      rpy="0 0 0"
+      xyz="0.0001 -0.0019 0.127"/>
+    <parent
+      link="$(arg robot_name)/link_3"/>
+    <child
+      link="$(arg robot_name)/link_4"/>
+    <dynamics
+      friction="0.1"
+      damping="0.1"/>
+  </joint>
   <link name="$(arg robot_name)/link_4">
-    <inertial>
-      <origin rpy="0 0 0" xyz="0.0 0.0 0"/>
-      <mass value="0.1" />
-      <inertia ixx="0.0" iyy="0.0" izz="0.0" ixy="-0.0" ixz="0" iyz="0" />
-    </inertial>
+    <visual>
+      <origin
+        rpy="0 0 0"
+        xyz="0 0 0"/>
+      <geometry>
+        <mesh
+          filename="${mesh_directory}/link_4.stl"
+          scale="1 1 1"/>
+      </geometry>
+      <material name="interbotix_black"/>
+    </visual>
+    <inertial>
+      <origin
+        rpy="0 0 0"
+        xyz="0.0 0.0 0"/>
+      <mass value="0.1"/>
+      <inertia
+        ixx="0.0"
+        iyy="0.0"
+        izz="0.0"
+        ixy="0.0"
+        ixz="0"
+        iyz="0"/>
+    </inertial>
+    <collision>
+      <origin
+        rpy="0 0 0"
+        xyz="0 0 0"/>
+      <geometry>
+        <mesh
+          filename="${mesh_directory}/link_4.stl"
+          scale="1 1 1"/>
+      </geometry>
+      <material name="interbotix_black"/>
+    </collision>
   </link>
  <joint name="j5" type="revolute">
     <axis xyz="0 0 1"/>
-    <limit effort="10" lower="${-pi + pi_offset}" upper="${pi - pi_offset}" velocity="${pi}"/>
-    <!-- <limit effort="5" lower="${radians(-122)}" upper="${radians(90)}" velocity="${pi}"/> -->
-    <origin rpy="0 0 0" xyz="0 0.03021 0.02761"/>
-    <parent link="$(arg robot_name)/link_4"/>
-    <child link="$(arg robot_name)/link_5"/>
-    <dynamics friction="0.1"/>
-  </joint>
-  <transmission name="trans_wrist_angle">
-    <type>transmission_interface/SimpleTransmission</type>
-    <joint name="j5">
-      <hardwareInterface>hardware_interface/EffortJointInterface</hardwareInterface>
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
Commit message: [xscobot_descriptions] Further refine URDF
Fix incorrect axis spec on some joints. Fix incorrect rotation of some
joints. Add fixed pseudo-joint between gripper_link and fingers_link to
prevent fingers from spinning.

File: interbotix_ros_xscobots/interbotix_xscobot_descriptions/urdf/dx400.urdf.xacro (robot description, xacro)
@@ -85,5 +85,5 @@
       velocity="${pi}"/>
     <origin
-      rpy="0 0 0"
+      rpy="0 0 ${pi/2}"
       xyz="0 0 0"/>
     <parent
@@ -133,5 +133,5 @@
   </link>
   <joint name="j2" type="revolute">
-    <axis xyz="0 1 0"/>
+    <axis xyz="0 -1 0"/>
     <limit
       effort="10"
@@ -188,5 +188,5 @@
   </link>
   <joint name="j3" type="revolute">
-    <axis xyz="0 1 0"/>
+    <axis xyz="0 -1 0"/>
     <limit
       effort="10"
@@ -360,5 +360,5 @@
       velocity="${pi}"/>
     <origin
-      rpy="0 0 0"
+      rpy="${pi/2} 0 0"
       xyz="0.04725 0 0.02305"/>
     <parent
@@ -420,7 +420,7 @@
       link="$(arg robot_name)/gripper_link"/>
     <child
-      link="$(arg robot_name)/fingers_link"/>
-  </joint>
-  <link name="$(arg robot_name)/fingers_link">
+      link="$(arg robot_name)/gripper_pinion_link"/>
+  </joint>
+  <link name="$(arg robot_name)/gripper_pinion_link">
     <inertial>
       <origin
@@ -437,34 +437,14 @@
     </inertial>
   </link>
-  <joint name="left_finger" type="prismatic">
-    <axis xyz="0 0 1"/>
-    <limit
-      effort="5"
-      lower="0.001"
-      upper="0.025"
-      velocity="1"/>
-    <origin
-      rpy="0 0 0"
-      xyz="0 0.01755 0"/>
-    <parent
+  <joint name="fingers_joint" type="fixed">
+    <origin
+      rpy="0 0 0"
+      xyz="0.046501 0 -0.024"/>
+    <parent
+      link="$(arg robot_name)/gripper_link"/>
+    <child
       link="$(arg robot_name)/fingers_link"/>
-    <child
-      link="$(arg robot_name)/left_finger_link"/>
-    <dynamics
-      friction="0.1"
-      damping="0.1"/>
-  </joint>
-  <link name="$(arg robot_name)/left_finger_link">
-    <visual>
-      <origin
-        rpy="0 0 0"
-        xyz="0 0 0"/>
-      <geometry>
-        <mesh
-          filename="${mesh_directory}/gripper_finger.stl"
-          scale="1 1 1"/>
-      </geometry>
-      <material name="interbotix_black"/>
-    </visual>
+  </joint>
+  <link name="$(arg robot_name)/fingers_link">
     <inertial>
       <origin
@@ -480,38 +460,27 @@
         iyz="0"/>
     </inertial>
-    <collision>
-      <origin
-        rpy="0 0 0"
-        xyz="0 0 0"/>
-      <geometry>
-        <mesh
-          filename="${mesh_directory}/gripper_finger.stl"
-          scale="1 1 1"/>
-      </geometry>
-      <material name="interbotix_black"/>
-    </collision>
-  </link>
-  <joint name="right_finger" type="prismatic">
+  </link>
+  <joint name="left_finger" type="prismatic">
     <axis xyz="0 0 1"/>
     <limit
       effort="5"
-      lower="-0.025"
-      upper="-0.001"
+      lower="0.001"
+      upper="0.025"
       velocity="1"/>
     <origin
       rpy="0 0 0"
-      xyz="0 -0.01755 0"/>
+      xyz="0 0.01755 0"/>
     <parent
       link="$(arg robot_name)/fingers_link"/>
     <child
-      link="$(arg robot_name)/right_finger_link"/>
-    <dynamics
-      friction="0.1"
-      damping="0.1"/>
-  </joint>
-  <link name="$(arg robot_name)/right_finger_link">
-    <visual>
-      <origin
-        rpy="${pi} 0 0"
+      link="$(arg robot_name)/left_finger_link"/>
+    <dynamics
+      friction="0.1"
+      damping="0.1"/>
+  </joint>
+  <link name="$(arg robot_name)/left_finger_link">
+    <visual>
+      <origin
+        rpy="0 0 0"
         xyz="0 0 0"/>
       <geometry>
@@ -537,4 +506,59 @@
     <collision>
       <origin
+        rpy="0 0 0"
+        xyz="0 0 0"/>
+      <geometry>
+        <mesh
+          filename="${mesh_directory}/gripper_finger.stl"
+          scale="1 1 1"/>
+      </geometry>
+      <material name="interbotix_black"/>
+    </collision>
+  </link>
+  <joint name="right_finger" type="prismatic">
+    <axis xyz="0 0 1"/>
+    <limit
+      effort="5"
+      lower="-0.025"
+      upper="-0.001"
+      velocity="1"/>
+    <origin
+      rpy="0 0 0"
+      xyz="0 -0.01755 0"/>
+    <parent
+      link="$(arg robot_name)/fingers_link"/>
+    <child
+      link="$(arg robot_name)/right_finger_link"/>
+    <dynamics
+      friction="0.1"
+      damping="0.1"/>
+  </joint>
+  <link name="$(arg robot_name)/right_finger_link">
+    <visual>
+      <origin
+        rpy="${pi} 0 0"
+        xyz="0 0 0"/>
+      <geometry>
+        <mesh
+          filename="${mesh_directory}/gripper_finger.stl"
+          scale="1 1 1"/>
+      </geometry>
+      <material name="interbotix_black"/>
+    </visual>
+    <inertial>
+      <origin
+        rpy="0 0 0"
+        xyz="0 0 0"/>
+      <mass value="0"/>
+      <inertia
+        ixx="0"
+        iyy="0"
+        izz="0"
+        ixy="0"
+        ixz="0"
+        iyz="0"/>
+    </inertial>
+    <collision>
+      <origin
         rpy="${pi} 0 0"
         xyz="0 0 0"/>

Commit message: [URDF] Fixed linting

File: interbotix_ros_xscobots/interbotix_xscobot_descriptions/urdf/dx400.urdf.xacro (robot description, xacro)
@@ -25,16 +25,16 @@
   <xacro:property name="hardware_type"    value="$(arg hardware_type)"/>
   <xacro:property name="pi_offset"        value="0.00001"/>
-  <xacro:property name="j1_limit_lower"        value="-6.70001"/>
-  <xacro:property name="j1_limit_upper"        value="0.00001"/>
-  <xacro:property name="j2_limit_lower"        value="-1.88001"/>
-  <xacro:property name="j2_limit_upper"        value="1.88001"/>
-  <xacro:property name="j3_limit_lower"        value="-2.70001"/>
-  <xacro:property name="j3_limit_upper"        value="2.70001"/>
-  <xacro:property name="j4_limit_lower"        value="-3.66001"/>
-  <xacro:property name="j4_limit_upper"        value="1.55001"/>
-  <xacro:property name="j5_limit_lower"        value="-4.00001"/>
-  <xacro:property name="j5_limit_upper"        value="1.60001"/>
-  <xacro:property name="j6_limit_lower"        value="-5.00001"/>
-  <xacro:property name="j6_limit_upper"        value="1.60001"/>
+  <xacro:property name="j1_limit_lower"   value="-6.70001"/>
+  <xacro:property name="j1_limit_upper"   value="0.00001"/>
+  <xacro:property name="j2_limit_lower"   value="-1.88001"/>
+  <xacro:property name="j2_limit_upper"   value="1.88001"/>
+  <xacro:property name="j3_limit_lower"   value="-2.70001"/>
+  <xacro:property name="j3_limit_upper"   value="2.70001"/>
+  <xacro:property name="j4_limit_lower"   value="-3.66001"/>
+  <xacro:property name="j4_limit_upper"   value="1.55001"/>
+  <xacro:property name="j5_limit_lower"   value="-4.00001"/>
+  <xacro:property name="j5_limit_upper"   value="1.60001"/>
+  <xacro:property name="j6_limit_lower"   value="-5.00001"/>
+  <xacro:property name="j6_limit_upper"   value="1.60001"/>
   <xacro:if value="$(arg load_gazebo_configs)">
     <xacro:include filename="$(find interbotix_common_sim)/textures/interbotix_texture.gazebo"/>

Commit message: [URDF] Rounded off joint limits

File: interbotix_ros_xscobots/interbotix_xscobot_descriptions/urdf/dx400.urdf.xacro (robot description, xacro)
@@ -24,17 +24,17 @@
   <xacro:property name="urdf_loc"         value="$(arg external_urdf_loc)"/>
   <xacro:property name="hardware_type"    value="$(arg hardware_type)"/>
-  <xacro:property name="pi_offset"        value="0.00001"/>
-  <xacro:property name="j1_limit_lower"   value="-6.70001"/>
-  <xacro:property name="j1_limit_upper"   value="0.00001"/>
-  <xacro:property name="j2_limit_lower"   value="-1.88001"/>
-  <xacro:property name="j2_limit_upper"   value="1.88001"/>
-  <xacro:property name="j3_limit_lower"   value="-2.70001"/>
-  <xacro:property name="j3_limit_upper"   value="2.70001"/>
-  <xacro:property name="j4_limit_lower"   value="-3.66001"/>
-  <xacro:property name="j4_limit_upper"   value="1.55001"/>
-  <xacro:property name="j5_limit_lower"   value="-4.00001"/>
-  <xacro:property name="j5_limit_upper"   value="1.60001"/>
-  <xacro:property name="j6_limit_lower"   value="-5.00001"/>
-  <xacro:property name="j6_limit_upper"   value="1.60001"/>
+  <xacro:property name="pi_offset"        value="0.00"/>
+  <xacro:property name="j1_limit_lower"   value="-6.7"/>
+  <xacro:property name="j1_limit_upper"   value="0.00"/>
+  <xacro:property name="j2_limit_lower"   value="-1.88"/>
+  <xacro:property name="j2_limit_upper"   value="1.88"/>
+  <xacro:property name="j3_limit_lower"   value="-2.70"/>
+  <xacro:property name="j3_limit_upper"   value="2.70"/>
+  <xacro:property name="j4_limit_lower"   value="-3.66"/>
+  <xacro:property name="j4_limit_upper"   value="1.55"/>
+  <xacro:property name="j5_limit_lower"   value="-4.00"/>
+  <xacro:property name="j5_limit_upper"   value="1.60"/>
+  <xacro:property name="j6_limit_lower"   value="-5.00"/>
+  <xacro:property name="j6_limit_upper"   value="1.60"/>
   <xacro:if value="$(arg load_gazebo_configs)">
     <xacro:include filename="$(find interbotix_common_sim)/textures/interbotix_texture.gazebo"/>

Commit message: Fixed errors and issues

File: interbotix_ros_xscobots/interbotix_xscobot_descriptions/urdf/dx400.urdf.xacro (robot description, xacro)
@@ -15,5 +15,4 @@
   <xacro:arg name="gripper_limit_max"     default="0.008"/>
   <xacro:arg name="show_ar_tag"           default="false"/>
-  <xacro:arg name="show_gripper_bar"      default="true"/>
   <xacro:arg name="show_gripper_fingers"  default="true"/>
   <xacro:arg name="use_world_frame"       default="false"/>
@@ -24,5 +23,5 @@
   <xacro:property name="urdf_loc"         value="$(arg external_urdf_loc)"/>
   <xacro:property name="hardware_type"    value="$(arg hardware_type)"/>
-  <xacro:property name="pi_offset"        value="0.00"/>
+  <xacro:property name="pi_offset"        value="0.00001"/>
   <xacro:property name="j1_limit_lower"   value="-6.7"/>
   <xacro:property name="j1_limit_upper"   value="0.00"/>

Commit message: [URDF] Fixed URDF Errors

File: interbotix_ros_xscobots/interbotix_xscobot_descriptions/urdf/dx400.urdf.xacro (robot description, xacro)
@@ -310,5 +310,5 @@
   </link>
  <joint name="j5" type="revolute">
-    <axis xyz="0 0 1"/>
+    <axis xyz="0 0 -1"/>
     <limit
       effort="10"
@@ -427,5 +427,5 @@
       velocity="${pi/2}"/>
     <origin
-      rpy="0 0 0"
+      rpy="${pi} 0 0"
       xyz="0.046501 0 -0.024"/>
     <parent
