Commit message: Updated URDF for bug fix

File: interbotix_ros_xscobots/interbotix_xscobot_descriptions/urdf/dx400.urdf.xacro (robot description, xacro)
@@ -545,4 +545,10 @@
       friction="0.1"
       damping="0.1"/>
+    <xacro:if value="${hardware_type != 'gz_classic'}">
+      <mimic
+        joint="left_finger"
+        multiplier="-1"
+        offset="0"/>
+    </xacro:if>
   </joint>
   <link name="$(arg robot_name)/right_finger_link">

Commit message: [xscobot_descriptions] Add ee_gripper_link
Adds the ee_gripper joint and ee_gripper_link link to the dx400 URDF.

File: interbotix_ros_xscobots/interbotix_xscobot_descriptions/urdf/dx400.urdf.xacro (robot description, xacro)
@@ -473,4 +473,26 @@
     </inertial>
   </link>
+  <joint name="ee_gripper" type="fixed">
+    <axis xyz="1 0 0"/>
+    <origin
+      rpy="0 0 0"
+      xyz="0.03 0 0"/>
+    <parent
+      link="$(arg robot_name)/fingers_link"/>
+    <child
+      link="$(arg robot_name)/ee_gripper_link"/>
+  </joint>
+  <link name="$(arg robot_name)/ee_gripper_link">
+    <inertial>
+      <mass value="0.001"/>
+      <inertia
+        ixx="0.001"
+        iyy="0.001"
+        izz="0.001"
+        ixy="0"
+        ixz="0"
+        iyz="0"/>
+    </inertial>
+  </link>
   <joint name="left_finger" type="prismatic">
     <axis xyz="0 0 1"/>

Commit message: Added gripper control fixes

File: interbotix_ros_xscobots/interbotix_xscobot_descriptions/urdf/dx400.urdf.xacro (robot description, xacro)
@@ -423,5 +423,5 @@
     <limit
       effort="1"
-      lower="0.0"
+      lower="-3.9"
       upper="3.9"
       velocity="${pi/2}"/>
@@ -505,5 +505,5 @@
       effort="5"
       lower="0.001"
-      upper="0.025"
+      upper="0.035"
       velocity="1.0"/>
     <origin
@@ -559,5 +559,5 @@
     <limit
       effort="5"
-      lower="-0.025"
+      lower="-0.035"
       upper="-0.001"
       velocity="1.0"/>

File: interbotix_ros_xscobots/interbotix_xscobot_moveit/config/srdf/dx400.srdf.xacro (robot description, xacro)
@@ -71,6 +71,6 @@
     <group_state name="open" group="interbotix_gripper">
         <!-- <joint name="gripper" value="2.05"/> -->
-        <joint name="left_finger" value="0.024"/>
-        <joint name="right_finger" value="-0.024"/>
+        <joint name="left_finger" value="0.035"/>
+        <joint name="right_finger" value="-0.035"/>
     </group_state>
     <group_state name="close" group="interbotix_gripper">

Commit message: Changes for ar tag

File: interbotix_ros_xscobots/interbotix_xscobot_descriptions/urdf/dx400.urdf.xacro (robot description, xacro)
@@ -614,5 +614,5 @@
   <xacro:if value="$(arg show_ar_tag)">
     <xacro:include filename="$(find interbotix_xscobot_descriptions)/urdf/ar_tag.urdf.xacro"/>
-  </xacro:if> <!-- show_ar_tag -->
+  </xacro:if>
   <xacro:if value="${urdf_loc != ''}">
     <xacro:include filename="${urdf_loc}"/>

File: interbotix_ros_xscobots/interbotix_xscobot_moveit/config/srdf/dx400.srdf.xacro (robot description, xacro)
@@ -47,11 +47,11 @@
     <group_state name="open" group="interbotix_gripper">
         <!-- <joint name="gripper" value="2.05"/> -->
-        <joint name="left_finger" value="0.035"/>
-        <joint name="right_finger" value="-0.035"/>
+        <joint name="left_finger" value="0.045"/>
+        <joint name="right_finger" value="-0.045"/>
     </group_state>
     <group_state name="close" group="interbotix_gripper">
         <!-- <joint name="gripper" value="0.05"/> -->
-        <joint name="left_finger" value="0.001"/>
-        <joint name="right_finger" value="-0.001"/>
+        <joint name="left_finger" value="0.00001"/>
+        <joint name="right_finger" value="-0.00001"/>
     </group_state>
     <!--END EFFECTOR: Purpose: Represent information about an end effector.-->
@@ -74,4 +74,13 @@
     <disable_collisions link1="$(arg robot_name)/link_4" link2="$(arg robot_name)/right_finger_link" reason="Never"/>
     <disable_collisions link1="$(arg robot_name)/link_5" link2="$(arg robot_name)/right_finger_link" reason="Never"/>
+    <xacro:if value="$(arg show_ar_tag)">
+      <disable_collisions link1="$(arg robot_name)/ar_tag_link" link2="$(arg robot_name)/right_finger_link" reason="Adjacent" />
+      <disable_collisions link1="$(arg robot_name)/ar_tag_link" link2="$(arg robot_name)/ar_tag_target_link" reason="Adjacent" />
+      <disable_collisions link1="$(arg robot_name)/ar_tag_link" link2="$(arg robot_name)/ee_gripper_link" reason="Adjacent" />
+      <disable_collisions link1="$(arg robot_name)/ar_tag_link" link2="$(arg robot_name)/left_finger_link" reason="Adjacent" />
+      <disable_collisions link1="$(arg robot_name)/ar_tag_link" link2="$(arg robot_name)/left_finger_link" reason="Adjacent" />
+      <disable_collisions link1="$(arg robot_name)/ar_tag_target_link" link2="$(arg robot_name)/right_finger_link" reason="Adjacent" />
+      <disable_collisions link1="$(arg robot_name)/ar_tag_target_link" link2="$(arg robot_name)/ee_gripper_link" reason="Adjacent" />
+    </xacro:if>
     <xacro:if value="${srdf_loc != ''}">
         <xacro:include filename="${srdf_loc}"/>

Commit message: Feature: moveit interface examples (#131)
* Fixed URDF nd SRDF

* Fixed and added YAML and Rviz Files

* Updated Launch file

* Added moveit python interface examples

* Fixed gripper calib issue

* Removed commented code

* Resolved suggested changes

* Added gripper control fixes

* [xscobot_descriptions] Add AR tag

* Added new line

* more fixes

* Update interbotix_ros_xscobots/interbotix_xscobot_descriptions/urdf/dx400.urdf.xacro

Co-authored-by: LSinterbotix <85308904+LSinterbotix@users.noreply.github.com>

* Update interbotix_ros_xscobots/interbotix_xscobot_moveit/CMakeLists.txt

Co-authored-by: LSinterbotix <85308904+LSinterbotix@users.noreply.github.com>

* Update interbotix_ros_xscobots/interbotix_xscobot_moveit/scripts/interbotix_moveit_example.py

Co-authored-by: LSinterbotix <85308904+LSinterbotix@users.noreply.github.com>

* Update interbotix_ros_xscobots/interbotix_xscobot_moveit/scripts/interbotix_moveit_example.py

Co-authored-by: LSinterbotix <85308904+LSinterbotix@users.noreply.github.com>

* Reverted test updates

* Update interbotix_ros_xscobots/interbotix_xscobot_moveit/launch/moveit_api.launch.py

Co-authored-by: LSinterbotix <85308904+LSinterbotix@users.noreply.github.com>

* Update interbotix_ros_xscobots/interbotix_xscobot_moveit/launch/moveit_api.launch.py

Co-authored-by: LSinterbotix <85308904+LSinterbotix@users.noreply.github.com>

* Update interbotix_ros_xscobots/interbotix_xscobot_moveit/launch/moveit_api.launch.py

Co-authored-by: LSinterbotix <85308904+LSinterbotix@users.noreply.github.com>

* [MoveIt_API]Fixed suggested changes

* [Cmake] Updated Cmakelist and package name

* Changes for ar tag

* Update interbotix_ros_xscobots/interbotix_xscobot_moveit/launch/xscobot_moveit.launch.py

Co-authored-by: LSinterbotix <85308904+LSinterbotix@users.noreply.github.com>

* Added docstring and removed unnecessary code.

* minor fixes

* Fixed lint

* fixed flake8 linting

* Update interbotix_ros_xscobots/interbotix_xscobot_moveit/demos/example.py

Co-authored-by: LSinterbotix <85308904+LSinterbotix@users.noreply.github.com>

* Fixed linting and compatibility

* [AR_TAG] Changes for added ar_tag

* Update interbotix_ros_xscobots/interbotix_xscobot_moveit/launch/moveit_api.launch.py

Co-authored-by: LSinterbotix <85308904+LSinterbotix@users.noreply.github.com>

* Update interbotix_ros_xscobots/interbotix_xscobot_moveit/launch/moveit_api.launch.py

Co-authored-by: LSinterbotix <85308904+LSinterbotix@users.noreply.github.com>

* Minor fixes

---------

Co-authored-by: Luke Schmitt <luke@trossenrobotics.com>
Co-authored-by: LSinterbotix <85308904+LSinterbotix@users.noreply.github.com>

File: interbotix_ros_xscobots/interbotix_xscobot_descriptions/urdf/dx400.urdf.xacro (robot description, xacro)
@@ -423,5 +423,5 @@
     <limit
       effort="1"
-      lower="0.0"
+      lower="-3.9"
       upper="3.9"
       velocity="${pi/2}"/>
@@ -500,5 +500,5 @@
       effort="5"
       lower="0.001"
-      upper="0.025"
+      upper="0.035"
       velocity="1.0"/>
     <origin
@@ -554,5 +554,5 @@
     <limit
       effort="5"
-      lower="-0.025"
+      lower="-0.035"
       upper="-0.001"
       velocity="1.0"/>
@@ -614,5 +614,5 @@
   <xacro:if value="$(arg show_ar_tag)">
     <xacro:include filename="$(find interbotix_xscobot_descriptions)/urdf/ar_tag.urdf.xacro"/>
-  </xacro:if> <!-- show_ar_tag -->
+  </xacro:if>
   <xacro:if value="${urdf_loc != ''}">
     <xacro:include filename="${urdf_loc}"/>

File: interbotix_ros_xscobots/interbotix_xscobot_moveit/config/srdf/dx400.srdf.xacro (robot description, xacro)
@@ -13,4 +13,5 @@
     <xacro:arg name="base_link_frame" default="base_link"/>
     <xacro:arg name="external_srdf_loc" default=""/>
+    <xacro:arg name="show_ar_tag" default="false"/>
     <xacro:property name="srdf_loc" value="$(arg external_srdf_loc)"/>
     <group name="interbotix_arm">
@@ -29,11 +30,35 @@
     </group>
     <!--GROUP STATES: Purpose: Define a named state for a particular group, in terms of joint values. This is useful to define states like 'folded arms'-->
+    <group_state name="pose1" group="interbotix_arm">
+        <joint name="j1" value="-1.3529"/>
+        <joint name="j2" value="1.7901"/>
+        <joint name="j3" value="-1.1949"/>
+        <joint name="j4" value="0.2239"/>
+        <joint name="j5" value="0.2669"/>
+        <joint name="j6" value="-0.1073"/>
+    </group_state>
+    <group_state name="pose2" group="interbotix_arm">
+        <joint name="j1" value="-0.688"/>
+        <joint name="j2" value="1.362"/>
+        <joint name="j3" value="-0.894"/>
+        <joint name="j4" value="-1.764"/>
+        <joint name="j5" value="-0.7531"/>
+        <joint name="j6" value="-0.7102"/>
+    </group_state>
+    <group_state name="pose3" group="interbotix_arm">
+        <joint name="j1" value="-0.2009"/>
+        <joint name="j2" value="1.9389"/>
+        <joint name="j3" value="-0.7700"/>
+        <joint name="j4" value="-0.7915"/>
+        <joint name="j5" value="0.1089"/>
+        <joint name="j6" value="-1.2225"/>
+    </group_state>
     <group_state name="sleep" group="interbotix_arm">
-        <joint name="j1" value="0.00"/>
+        <joint name="j1" value="-1.57"/>
         <joint name="j2" value="2.00"/>
         <joint name="j3" value="-2.83"/>
         <joint name="j4" value="-2.46"/>
         <joint name="j5" value="0.0"/>
-        <joint name="j6" value="-1.7"/>
+        <joint name="j6" value="-1.57"/>
     </group_state>
     <group_state name="home" group="interbotix_arm">
@@ -47,11 +72,11 @@
     <group_state name="open" group="interbotix_gripper">
         <!-- <joint name="gripper" value="2.05"/> -->
-        <joint name="left_finger" value="0.024"/>
-        <joint name="right_finger" value="-0.024"/>
+        <joint name="left_finger" value="0.045"/>
+        <joint name="right_finger" value="-0.045"/>
     </group_state>
     <group_state name="close" group="interbotix_gripper">
         <!-- <joint name="gripper" value="0.05"/> -->
-        <joint name="left_finger" value="0.001"/>
-        <joint name="right_finger" value="-0.001"/>
+        <joint name="left_finger" value="0.00001"/>
+        <joint name="right_finger" value="-0.00001"/>
     </group_state>
     <!--END EFFECTOR: Purpose: Represent information about an end effector.-->
@@ -74,4 +99,13 @@
     <disable_collisions link1="$(arg robot_name)/link_4" link2="$(arg robot_name)/right_finger_link" reason="Never"/>
     <disable_collisions link1="$(arg robot_name)/link_5" link2="$(arg robot_name)/right_finger_link" reason="Never"/>
+    <xacro:if value="$(arg show_ar_tag)">
+      <disable_collisions link1="$(arg robot_name)/ar_tag_link" link2="$(arg robot_name)/right_finger_link" reason="Adjacent" />
+      <disable_collisions link1="$(arg robot_name)/ar_tag_link" link2="$(arg robot_name)/ar_tag_target_link" reason="Adjacent" />
+      <disable_collisions link1="$(arg robot_name)/ar_tag_link" link2="$(arg robot_name)/ee_gripper_link" reason="Adjacent" />
+      <disable_collisions link1="$(arg robot_name)/ar_tag_link" link2="$(arg robot_name)/left_finger_link" reason="Adjacent" />
+      <disable_collisions link1="$(arg robot_name)/ar_tag_link" link2="$(arg robot_name)/left_finger_link" reason="Adjacent" />
+      <disable_collisions link1="$(arg robot_name)/ar_tag_target_link" link2="$(arg robot_name)/right_finger_link" reason="Adjacent" />
+      <disable_collisions link1="$(arg robot_name)/ar_tag_target_link" link2="$(arg robot_name)/ee_gripper_link" reason="Adjacent" />
+    </xacro:if>
     <xacro:if value="${srdf_loc != ''}">
         <xacro:include filename="${srdf_loc}"/>
