Commit message: [SRDF] Changed group name, added robot_name param

File: interbotix_ros_xscobots/interbotix_xscobot_moveit/config/srdf/dx400.srdf.xacro (robot description, xacro)
@@ -14,5 +14,5 @@
     <xacro:arg name="external_srdf_loc" default=""/>
     <xacro:property name="srdf_loc" value="$(arg external_srdf_loc)"/>
-    <group name="dx400">
+    <group name="interbotix_arm">
         <joint name="virtual_joint"/>
         <joint name="j1"/>
@@ -23,12 +23,12 @@
         <joint name="j6"/>
     </group>
-    <group name="hand">
-        <link name="dx400/fingers_link"/>
-        <link name="dx400/left_finger_link"/>
-        <link name="dx400/right_finger_link"/>
-        <link name="dx400/gripper_pinion_link"/>
+    <group name="interbotix_gripper">
+        <link name="$(arg robot_name)/fingers_link"/>
+        <link name="$(arg robot_name)/left_finger_link"/>
+        <link name="$(arg robot_name)/right_finger_link"/>
+        <link name="$(arg robot_name)/gripper_pinion_link"/>
     </group>
     <!--GROUP STATES: Purpose: Define a named state for a particular group, in terms of joint values. This is useful to define states like 'folded arms'-->
-    <group_state name="home" group="dx400">
+    <group_state name="home" group="interbotix_arm">
         <joint name="j1" value="0"/>
         <joint name="j2" value="0"/>
@@ -38,10 +38,10 @@
         <joint name="j6" value="0"/>
     </group_state>
-    <group_state name="open" group="hand">
+    <group_state name="open" group="interbotix_gripper">
         <joint name="gripper" value="0"/>
         <joint name="left_finger" value="0.024"/>
         <joint name="right_finger" value="-0.024"/>
     </group_state>
-    <group_state name="close" group="hand">
+    <group_state name="close" group="interbotix_gripper">
         <joint name="gripper" value="0"/>
         <joint name="left_finger" value="0.001"/>
@@ -49,22 +49,22 @@
     </group_state>
     <!--END EFFECTOR: Purpose: Represent information about an end effector.-->
-    <end_effector name="hand" parent_link="dx400/gripper_link" group="dx400"/>
+    <end_effector name="interbotix_gripper" parent_link="$(arg robot_name)/gripper_link" group="interbotix_arm"/>
     <!--VIRTUAL JOINT: Purpose: this element defines a virtual joint between a robot link and an external frame of reference (considered fixed with respect to the robot)-->
-    <virtual_joint name="virtual_joint" type="fixed" parent_frame="world" child_link="dx400/base_link"/>
+    <virtual_joint name="virtual_joint" type="fixed" parent_frame="world" child_link="$(arg robot_name)/base_link"/>
     <!--DISABLE COLLISIONS: By default it is assumed that any link of the robot could potentially come into collision with any other link in the robot. This tag disables collision checking between a specified pair of links. -->
-    <disable_collisions link1="dx400/base_link" link2="dx400/link_1" reason="Adjacent"/>
-    <disable_collisions link1="dx400/gripper_link" link2="dx400/left_finger_link" reason="Adjacent"/>
-    <disable_collisions link1="dx400/gripper_link" link2="dx400/link_4" reason="Never"/>
-    <disable_collisions link1="dx400/gripper_link" link2="dx400/link_5" reason="Adjacent"/>
-    <disable_collisions link1="dx400/gripper_link" link2="dx400/right_finger_link" reason="Adjacent"/>
-    <disable_collisions link1="dx400/left_finger_link" link2="dx400/link_4" reason="Never"/>
-    <disable_collisions link1="dx400/left_finger_link" link2="dx400/link_5" reason="Never"/>
-    <disable_collisions link1="dx400/left_finger_link" link2="dx400/right_finger_link" reason="Adjacent"/>
-    <disable_collisions link1="dx400/link_1" link2="dx400/link_2" reason="Adjacent"/>
-    <disable_collisions link1="dx400/link_2" link2="dx400/link_3" reason="Adjacent"/>
-    <disable_collisions link1="dx400/link_3" link2="dx400/link_4" reason="Adjacent"/>
-    <disable_collisions link1="dx400/link_4" link2="dx400/link_5" reason="Adjacent"/>
-    <disable_collisions link1="dx400/link_4" link2="dx400/right_finger_link" reason="Never"/>
-    <disable_collisions link1="dx400/link_5" link2="dx400/right_finger_link" reason="Never"/>
+    <disable_collisions link1="$(arg robot_name)/base_link" link2="$(arg robot_name)/link_1" reason="Adjacent"/>
+    <disable_collisions link1="$(arg robot_name)/gripper_link" link2="$(arg robot_name)/left_finger_link" reason="Adjacent"/>
+    <disable_collisions link1="$(arg robot_name)/gripper_link" link2="$(arg robot_name)/link_4" reason="Never"/>
+    <disable_collisions link1="$(arg robot_name)/gripper_link" link2="$(arg robot_name)/link_5" reason="Adjacent"/>
+    <disable_collisions link1="$(arg robot_name)/gripper_link" link2="$(arg robot_name)/right_finger_link" reason="Adjacent"/>
+    <disable_collisions link1="$(arg robot_name)/left_finger_link" link2="$(arg robot_name)/link_4" reason="Never"/>
+    <disable_collisions link1="$(arg robot_name)/left_finger_link" link2="$(arg robot_name)/link_5" reason="Never"/>
+    <disable_collisions link1="$(arg robot_name)/left_finger_link" link2="$(arg robot_name)/right_finger_link" reason="Adjacent"/>
+    <disable_collisions link1="$(arg robot_name)/link_1" link2="$(arg robot_name)/link_2" reason="Adjacent"/>
+    <disable_collisions link1="$(arg robot_name)/link_2" link2="$(arg robot_name)/link_3" reason="Adjacent"/>
+    <disable_collisions link1="$(arg robot_name)/link_3" link2="$(arg robot_name)/link_4" reason="Adjacent"/>
+    <disable_collisions link1="$(arg robot_name)/link_4" link2="$(arg robot_name)/link_5" reason="Adjacent"/>
+    <disable_collisions link1="$(arg robot_name)/link_4" link2="$(arg robot_name)/right_finger_link" reason="Never"/>
+    <disable_collisions link1="$(arg robot_name)/link_5" link2="$(arg robot_name)/right_finger_link" reason="Never"/>
     <xacro:if value="${srdf_loc != ''}">
         <xacro:include filename="${srdf_loc}"/>

Commit message: [YAML] Added sleep positions

File: interbotix_ros_xscobots/interbotix_xscobot_moveit/config/srdf/dx400.srdf.xacro (robot description, xacro)
@@ -30,11 +30,19 @@
     </group>
     <!--GROUP STATES: Purpose: Define a named state for a particular group, in terms of joint values. This is useful to define states like 'folded arms'-->
+    <group_state name="sleep" group="interbotix_arm">
+        <joint name="j1" value="0.00"/>
+        <joint name="j2" value="2.00"/>
+        <joint name="j3" value="-2.83"/>
+        <joint name="j4" value="-2.46"/>
+        <joint name="j5" value="0.0"/>
+        <joint name="j6" value="-1.7"/>
+    </group_state>
     <group_state name="home" group="interbotix_arm">
-        <joint name="j1" value="0"/>
-        <joint name="j2" value="0"/>
-        <joint name="j3" value="0"/>
-        <joint name="j4" value="0"/>
-        <joint name="j5" value="0"/>
-        <joint name="j6" value="0"/>
+        <joint name="j1" value="0.00"/>
+        <joint name="j2" value="0.00"/>
+        <joint name="j3" value="0.00"/>
+        <joint name="j4" value="0.00"/>
+        <joint name="j5" value="0.00"/>
+        <joint name="j6" value="0.00"/>
     </group_state>
     <group_state name="open" group="interbotix_gripper">

Commit message: [SRDF] Updated SRDF for gripper control

File: interbotix_ros_xscobots/interbotix_xscobot_moveit/config/srdf/dx400.srdf.xacro (robot description, xacro)
@@ -24,8 +24,7 @@
     </group>
     <group name="interbotix_gripper">
-        <link name="$(arg robot_name)/fingers_link"/>
+        <!-- <joint name="gripper"/> -->
         <link name="$(arg robot_name)/left_finger_link"/>
         <link name="$(arg robot_name)/right_finger_link"/>
-        <link name="$(arg robot_name)/gripper_pinion_link"/>
     </group>
     <!--GROUP STATES: Purpose: Define a named state for a particular group, in terms of joint values. This is useful to define states like 'folded arms'-->
@@ -47,10 +46,10 @@
     </group_state>
     <group_state name="open" group="interbotix_gripper">
-        <joint name="gripper" value="0"/>
+        <!-- <joint name="gripper" value="2.05"/> -->
         <joint name="left_finger" value="0.024"/>
         <joint name="right_finger" value="-0.024"/>
     </group_state>
     <group_state name="close" group="interbotix_gripper">
-        <joint name="gripper" value="0"/>
+        <!-- <joint name="gripper" value="0.05"/> -->
         <joint name="left_finger" value="0.001"/>
         <joint name="right_finger" value="-0.001"/>

Commit message: more fixes

File: interbotix_ros_xscobots/interbotix_xscobot_moveit/config/srdf/dx400.srdf.xacro (robot description, xacro)
@@ -29,28 +29,4 @@
     </group>
     <!--GROUP STATES: Purpose: Define a named state for a particular group, in terms of joint values. This is useful to define states like 'folded arms'-->
-    <group_state name="pose1" group="interbotix_arm">
-        <joint name="j1" value="-0.945"/>
-        <joint name="j2" value="1.663"/>
-        <joint name="j3" value="-2.103"/>
-        <joint name="j4" value="-1.738"/>
-        <joint name="j5" value="0.242"/>
-        <joint name="j6" value="-2.368"/>
-    </group_state>
-    <group_state name="pose2" group="interbotix_arm">
-        <joint name="j1" value="2.839"/>
-        <joint name="j2" value="1.96"/>
-        <joint name="j3" value="-2.29"/>
-        <joint name="j4" value="-1.845"/>
-        <joint name="j5" value="-0.153"/>
-        <joint name="j6" value="1.618"/>
-    </group_state>
-    <group_state name="pose3" group="interbotix_arm">
-        <joint name="j1" value="-1.97"/>
-        <joint name="j2" value="1.668"/>
-        <joint name="j3" value="-2.404"/>
-        <joint name="j4" value="-0.983"/>
-        <joint name="j5" value="-0.228"/>
-        <joint name="j6" value="0.047"/>
-    </group_state>
     <group_state name="sleep" group="interbotix_arm">
         <joint name="j1" value="-1.57"/>

Commit message: [AR_TAG] Changes for added ar_tag

File: interbotix_ros_xscobots/interbotix_xscobot_moveit/config/srdf/dx400.srdf.xacro (robot description, xacro)
@@ -13,4 +13,5 @@
     <xacro:arg name="base_link_frame" default="base_link"/>
     <xacro:arg name="external_srdf_loc" default=""/>
+    <xacro:arg name="show_ar_tag" default="false"/>
     <xacro:property name="srdf_loc" value="$(arg external_srdf_loc)"/>
     <group name="interbotix_arm">
@@ -29,4 +30,28 @@
     </group>
     <!--GROUP STATES: Purpose: Define a named state for a particular group, in terms of joint values. This is useful to define states like 'folded arms'-->
+    <group_state name="pose1" group="interbotix_arm">
+        <joint name="j1" value="-1.3529"/>
+        <joint name="j2" value="1.7901"/>
+        <joint name="j3" value="-1.1949"/>
+        <joint name="j4" value="0.2239"/>
+        <joint name="j5" value="0.2669"/>
+        <joint name="j6" value="-0.1073"/>
+    </group_state>
+    <group_state name="pose2" group="interbotix_arm">
+        <joint name="j1" value="-0.688"/>
+        <joint name="j2" value="1.362"/>
+        <joint name="j3" value="-0.894"/>
+        <joint name="j4" value="-1.764"/>
+        <joint name="j5" value="-0.7531"/>
+        <joint name="j6" value="-0.7102"/>
+    </group_state>
+    <group_state name="pose3" group="interbotix_arm">
+        <joint name="j1" value="-0.2009"/>
+        <joint name="j2" value="1.9389"/>
+        <joint name="j3" value="-0.7700"/>
+        <joint name="j4" value="-0.7915"/>
+        <joint name="j5" value="0.1089"/>
+        <joint name="j6" value="-1.2225"/>
+    </group_state>
     <group_state name="sleep" group="interbotix_arm">
         <joint name="j1" value="-1.57"/>
